File: project/machine that draw.kicad_pcb (KiCad board)
At the start: 2 copper layers, 24 parts, among them J1 Moteur1, J11 Barrel_Jack_Switch, J12 BAU, J13 Conn_02x03_Odd_Even, J14 Conn_02x03_Odd_Even, J2 SW_Y, J3 SD_Card_Device, J6 SERVO, J7 OLED, J8 Moteur2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

Commit message: finalisation du pcb
Parts:
- removed SW1: SW_Push, makerspace-unilasalle:SW_Push_KMR2
- added C1: 10uF, Capacitor_SMD:C_1206_3216Metric_Pad1.33x1.80mm_HandSolder, F.Cu at (116.0, 55.2)
- added C3: 10uF, Capacitor_SMD:C_1206_3216Metric_Pad1.33x1.80mm_HandSolder, F.Cu at (116.0, 61.5)
- J14, J3: moved to F.Cu
- moved J7 80.1 mm to (115.4, 69.5)
- moved A1 74.3 mm to (111.8, 38.4), turned to -90 degrees
- moved A3 73.7 mm to (87.4, 38.4), turned to -90 degrees
- moved J1 71.7 mm to (106.7, 34.5), turned to -90 degrees
- moved J8 71.1 mm to (82.3, 34.7), turned to -90 degrees
- moved J13 64.7 mm to (101.6, 54.9), turned to -90 degrees
- moved J3 63.0 mm to (50.5, 61.2), turned to 0 degrees
- moved J14 60.0 mm to (77.2, 54.9), turned to -90 degrees
- moved J2 59.8 mm to (74.5, 61.5)
- moved U1 59.7 mm to (110.1, 26.2)
- moved J9 59.5 mm to (78.2, 61.5)
- moved J11 59.0 mm to (118.0, 31.4)
- moved J12 59.0 mm to (122.0, 41.2)
- moved R2 57.1 mm to (58.5, 43.0), turned to 180 degrees
- moved U3 55.5 mm to (120.4, 55.9), turned to -90 degrees
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Connections:
- J13 pad 1: Net-(A1-MS1) -> Net-(A1-MS3)
- J13 pad 5: Net-(A1-MS3) -> Net-(A1-MS1)
- J2 pad 1: +5V -> +3.3V
- J9 pad 1: +5V -> +3.3V
- U1 pad 25: DIR2 -> STEP2
- U1 pad 26: STEP2 -> DIR2
- U1 pad 27: DIR1 -> STEP1
- U1 pad 28: STEP1 -> DIR1
Routing:
- net +3.3V: track 0.00 -> 160.2 mm
- net MOSI: track 0.00 -> 110.4 mm
- net +12V: track 0.00 -> 102.3 mm
- net MISO: track 0.00 -> 70.8 mm
- net CS: track 0.00 -> 66.4 mm
- net ENABLE: track 0.00 -> 62.5 mm
- net SCK: track 0.00 -> 58.6 mm
- net +5V: track 0.00 -> 51.0 mm
- net STEP2: track 0.00 -> 33.9 mm
- net DIR2: track 0.00 -> 33.9 mm
- net DIR1: track 0.00 -> 26.8 mm
- net STEP1: track 0.00 -> 25.3 mm
- net SDA: track 0.00 -> 17.0 mm
- net SCL: track 0.00 -> 14.2 mm
- net Net-(J12-Pin_1): track 0.00 -> 11.4 mm
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- added copper zone on B.Cu, net GND
- added copper zone on F.Cu, net GND
Other:
- board outline added: 94 x 53 mm
- board text added: "Machine that draws Equipe 2 Solange, Raphaël, Camilia, Tristan, Ange"
